File: Whips-PCB/Whips-PCB.kicad_pcb (KiCad board)
At the start: 2 copper layers, 82 x 86 mm, 28 parts, among them J1 12 VDC, J2 RS422 BUS, J3 SPEAKER 4OHM, J4 TO WHIP, J5 RS422 BUS, SW2 SW_DIP_x06, U2 MAX485ESA+T, U3 SN74AHCT125DR, U4 TSR_1-2450, U5 MAX98357AETE+T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

Commit message: cute turtle logo
Parts:
- added H1: DNP (LOGO), Joels KiCad Footprint Library:Turtle-Art-2024, F.Cu at (96.5, 137.1)
- D1: renamed from RECEIVING POWER
- D2: renamed from RECEIVING DATA
Other:
- board text added: "DATA"
- board text added: "FUTURE TURTLES 2024 WHIP CONTROLLER v 1.0.000"
- board text added: "POWER"

Commit message: Much better turtle logo with backlights
Parts:
- added D3: LED, Joels KiCad Footprint Library:Everlight 99-218GLM2C-L7277SGU-TR8-T0-ES side view LED, B.Cu at (95.8, 133.7)
- added D4: LED, Joels KiCad Footprint Library:Everlight 99-218GLM2C-L7277SGU-TR8-T0-ES side view LED, B.Cu at (129.8, 133.6)
- added R10: 470, Resistor_SMD:R_0402_1005Metric, B.Cu at (94.2, 128.3)
- added R11: 470, Resistor_SMD:R_0402_1005Metric, B.Cu at (125.0, 128.3)
- moved H1 16.7 mm to (112.8, 133.3)
Routing:
- net +3.3V: track 70.1 -> 172.1 mm, vias 1 -> 3
- net Net-(D4-K): track 0.00 -> 10.7 mm
- net Net-(D3-K): track 0.00 -> 3.68 mm
- net /12VDC: track 116.9 -> 119.4 mm
- net +5V: track 112.7 -> 112.2 mm
- net GND: vias 9 -> 21
- added copper zone on F.Cu, net GND

Commit message: Latest PCBs and some new gitignore stuff
Parts:
- J1, J2, J3, J5: footprint TerminalBlock_RND:TerminalBlock_RND_205-00001_1x02_P5.00mm_Horizontal -> TerminalBlock_Phoenix:TerminalBlock_Phoenix_MKDS-1,5-2_1x02_P5.00mm_Horizontal
- J4: footprint TerminalBlock_RND:TerminalBlock_RND_205-00002_1x03_P5.00mm_Horizontal -> TerminalBlock_Phoenix:TerminalBlock_Phoenix_MKDS-1,5-3_1x03_P5.00mm_Horizontal
